File: hw/icbm_control/icbm_control.brd (EAGLE design)
At the start: 71.1 x 66 mm, 52 parts, among them Q2 FDN306P, Q3 8 MHz, U1 PIC24FV16KM202, U2 A4960, X1 ICD, X2 Console

Commit message: oldie sync
Parts:
- C1: device ch_passive:CAP_RAD_8MM -> ch_passive:CAP_RAD_8MM_TT
- D2: device ch_generic:LED5MM -> ch_generic:LED5MM_TT
- JP1: device ch_connectors:1X02 -> ch_connectors:1X02-LUT
- Q3: device ch_passive:HC49US -> ch_passive:HC49US_TT
- S1, S2: device ch_passive:TACTILE-PTH -> ch_passive:TACT_PTH-LUT
- U1: device ch_microchip:DIL28-3 -> ch_microchip:DIL28-3-TT
- moved JP1 1.27 mm to (57.8, 38.1)
- moved C8 0.32 mm to (54.0, 21.0)
- moved R1 0.32 mm to (50.8, 21.0)
Routing:
- added copper zone on layer 1, net GND
