File: hw/icbm_control/icbm_control.sch (EAGLE design)
At the start: 52 parts, among them Q2 FDN306P, Q3 8 MHz, U1 PIC24FV16KM202, U2 A4960, X1 ICD, X2 Console

Commit message: oldie sync
Parts:
- C1: device ch_passive:CAP_POL-RAD8 -> ch_passive:CAP_POL-RAD8-TT
- D2: device ch_generic:LED5MM -> ch_generic:LED-TT
- JP1: device ch_connectors:JP1EPTH -> ch_connectors:JP1E-LUT
- Q3: device ch_passive:CRYSTAL_SFEHC49US -> ch_passive:CRYSTAL_SFE-TT
- S1, S2: device ch_passive:TAC_SWITCHPTH -> ch_passive:TAC_SWITCH-LUT
- U1: device ch_microchip:PIC24FX16KM202-DIP -> ch_microchip:PIC24FX16KM202-TT

Commit message: diag output added on status
Connections:
- net MISO: now also U1.RB10/PGED2; no longer U1.PGED2
- net PWM: now also U1.OC5/SDI2/RA7; no longer U1.SDI2/RA7
- net SCLK: now also U1.RB11/PGEC2; no longer U1.PGEC2
- net TACHO: now also U1.RB12/AN12/IC3/DAC1OUT; no longer U1.RB12/AN12/OC2B/DAC1OUT
Changed lines of the file:
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@@
 <setting verticaltext="up"/>
 </settings>
-<grid distance="0.1" unitdist="inch" unit="inch" style="lines" multiple="1" display="no" altdistance="0.01" altunitdist="inch" altunit="inch"/>
+<grid distance="0.1" unitdist="inch" unit="inch" style="lines" multiple="1" display="yes" altdistance="0.01" altunitdist="inch" altunit="inch"/>
 <layers>
-<layer number="1" name="Top" color="4" fill="1" visible="yes" active="no"/>
-<layer number="2" name="Route2" color="1" fill="3" visible="yes" active="no"/>
-<layer number="3" name="Route3" color="4" fill="3" visible="yes" active="no"/>
-<layer number="4" name="Route4" color="1" fill="4" visible="yes" active="no"/>
-<layer number="5" name="Route5" color="4" fill="4" visible="yes" active="no"/>
-<layer number="6" name="Route6" color="1" fill="8" visible="yes" active="no"/>
-<layer number="7" name="Route7" color="4" fill="8" visible="yes" active="no"/>
-<layer number="8" name="Route8" color="1" fill="2" visible="yes" active="no"/>
-<layer number="9" name="Route9" color="4" fill="2" visible="yes" active="no"/>
-<layer number="10" name="Route10" color="1" fill="7" visible="yes" active="no"/>
-<layer number="11" name="Route11" color="4" fill="7" visible="yes" active="no"/>
-<layer number="12" name="Route12" color="1" fill="5" visible="yes" active="no"/>
-<layer number="13" name="Route13" color="4" fill="5" visible="yes" active="no"/>
-<layer number="14" name="Route14" color="1" fill="6" visible="yes" active="no"/>
-<layer number="15" name="Route15" color="4" fill="6" visible="yes" active="no"/>
-<layer number="16" name="Bottom" color="1" fill="1" visible="yes" active="no"/>
-<layer number="17" name="Pads" color="2" fill="1" visible="yes" active="no"/>
-<layer number="18" name="Vias" color="2" fill="1" visible="yes" active="no"/>
-<layer number="19" name="Unrouted" color="6" fill="1" visible="yes" active="no"/>
-<layer number="20" name="Dimension" color="15" fill="1" visible="yes" active="no"/>
-<layer number="21" name="tPlace" color="7" fill="1" visible="yes" active="no"/>
-<layer number="22" name="bPlace" color="7" fill="1" visible="yes" active="no"/>
-<layer number="23" name="tOrigins" color="15" fill="1" visible="yes" active="no"/>
-<layer number="24" name="bOrigins" color="15" fill="1" visible="yes" active="no"/>
-<layer number="25" name="tNames" color="7" fill="1" visible="yes" active="no"/>
-<layer number="26" name="bNames" color="7" fill="1" visible="yes" active="no"/>
-<layer number="27" name="tValues" color="7" fill="1" visible="yes" active="no"/>
-<layer number="28" name="bValues" color="7" fill="1" visible="yes" active="no"/>
+<layer number="1" name="Top" color="4" fill="1" visible="no" active="no"/>
+<layer number="2" name="Route2" color="1" fill="3" visible="no" active="no"/>
+<layer number="3" name="Route3" color="4" fill="3" visible="no" active="no"/>
+<layer number="4" name="Route4" color="1" fill="4" visible="no" active="no"/>
+<layer number="5" name="Route5" color="4" fill="4" visible="no" active="no"/>
+<layer number="6" name="Route6" color="1" fill="8" visible="no" active="no"/>
+<layer number="7" name="Route7" color="4" fill="8" visible="no" active="no"/>
+<layer number="8" name="Route8" color="1" fill="2" visible="no" active="no"/>
+<layer number="9" name="Route9" color="4" fill="2" visible="no" active="no"/>
+<layer number="10" name="Route10" color="1" fill="7" visible="no" active="no"/>
+<layer number="11" name="Route11" color="4" fill="7" visible="no" active="no"/>
+<layer number="12" name="Route12" color="1" fill="5" visible="no" active="no"/>
+<layer number="13" name="Route13" color="4" fill="5" visible="no" active="no"/>
+<layer number="14" name="Route14" color="1" fill="6" visible="no" active="no"/>
+<layer number="15" name="Route15" color="4" fill="6" visible="no" active="no"/>
+<layer number="16" name="Bottom" color="1" fill="1" visible="no" active="no"/>
+<layer number="17" name="Pads" color="2" fill="1" visible="no" active="no"/>
+<layer number="18" name="Vias" color="2" fill="1" visible="no" active="no"/>
+<layer number="19" name="Unrouted" color="6" fill="1" visible="no" active="no"/>
+<layer number="20" name="Dimension" color="15" fill="1" visible="no" active="no"/>
+<layer number="21" name="tPlace" color="7" fill="1" visible="no" active="no"/>
+<layer number="22" name="bPlace" color="7" fill="1" visible="no" active="no"/>
+<layer number="23" name="tOrigins" color="15" fill="1" visible="no" active="no"/>
+<layer number="24" name="bOrigins" color="15" fill="1" visible="no" active="no"/>
+<layer number="25" name="tNames" color="7" fill="1" visible="no" active="no"/>
+<layer number="26" name="bNames" color="7" fill="1" visible="no" active="no"/>
+<layer number="27" name="tValues" color="7" fill="1" visible="no" active="no"/>
+<layer number="28" name="bValues" color="7" fill="1" visible="no" active="no"/>
 <layer number="29" name="tStop" color="7" fill="3" visible="no" active="no"/>
 <layer number="30" name="bStop" color="7" fill="6" visible="no" active="no"/>
@@
 <layer number="35" name="tGlue" color="7" fill="4" visible="no" active="no"/>
 <layer number="36" name="bGlue" color="7" fill="5" visible="no" active="no"/>
-<layer number="37" name="tTest" color="7" fill="1" visible="yes" active="no"/>
-<layer number="38" name="bTest" color="7" fill="1" visible="yes" active="no"/>
+<layer number="37" name="tTest" color="7" fill="1" visible="no" active="no"/>
+<layer number="38" name="bTest" color="7" fill="1" visible="no" active="no"/>
 <layer number="39" name="tKeepout" color="4" fill="11" visible="no" active="no"/>
 <layer number="40" name="bKeepout" color="1" fill="11" visible="no" active="no"/>
@@
 <layer number="44" name="Drills" color="7" fill="1" visible="no" active="no"/>
 <layer number="45" name="Holes" color="7" fill="1" visible="no" active="no"/>
-<layer number="46" name="Milling" color="3" fill="1" visible="yes" active="no"/>
-<layer number="47" name="Measures" color="7" fill="1" visible="yes" active="no"/>
-<layer number="48" name="Document" color="7" fill="1" visible="yes" active="no"/>
-<layer number="49" name="Reference" color="7" fill="1" visible="yes" active="no"/>
-<layer number="50" name="dxf" color="7" fill="1" visible="yes" active="no"/>
-<layer number="51" name="tDocu" color="7" fill="1" visible="yes" active="no"/>
-<layer number="52" name="bDocu" color="7" fill="1" visible="yes" active="no"/>
-<layer number="53" name="tGND_GNDA" color="7" fill="9" visible="yes" active="no"/>
-<layer number="54" name="bGND_GNDA" color="1" fill="9" visible="yes" active="no"/>
-<layer number="56" name="wert" color="7" fill="1" visible="yes" active="no"/>
-<layer number="57" name="tCAD" color="7" fill="1" visible="yes" active="no"/>
-<layer number="59" name="tCarbon" color="7" fill="1" visible="yes" active="no"/>
-<layer number="60" name="bCarbon" color="7" fill="1" visible="yes" active="no"/>
+<layer number="46" name="Milling" color="3" fill="1" visible="no" active="no"/>
+<layer number="47" name="Measures" color="7" fill="1" visible="no" active="no"/>
+<layer number="48" name="Document" color="7" fill="1" visible="no" active="no"/>
+<layer number="49" name="Reference" color="7" fill="1" visible="no" active="no"/>
+<layer number="50" name="dxf" color="7" fill="1" visible="no" active="no"/>
+<layer number="51" name="tDocu" color="7" fill="1" visible="no" active="no"/>
+<layer number="52" name="bDocu" color="7" fill="1" visible="no" active="no"/>
+<layer number="53" name="tGND_GNDA" color="7" fill="9" visible="no" active="no"/>
+<layer number="54" name="bGND_GNDA" color="1" fill="9" visible="no" active="no"/>
+<layer number="56" name="wert" color="7" fill="1" visible="no" active="no"/>
+<layer number="57" name="tCAD" color="7" fill="1" visible="no" active="no"/>
+<layer number="59" name="tCarbon" color="7" fill="1" visible="no" active="no"/>
+<layer number="60" name="bCarbon" color="7" fill="1" visible="no" active="no"/>
 <layer number="90" name="Modules" color="5" fill="1" visible="yes" active="yes"/>
 <layer number="91" name="Nets" color="2" fill="1" visible="yes" active="yes"/>
@@
 </segment>
 <segment>
-<pinref part="U1" gate="G$1" pin="PGED2"/>
+<pinref part="U1" gate="G$1" pin="RB10/PGED2"/>
 <wire x1="83.82" y1="208.28" x2="86.36" y2="208.28" width="0.1524" layer="91"/>
 <label x="76.2" y="208.28" size="1.778" layer="95"/>
@@
 </segment>
 <segment>
-<pinref part="U1" gate="G$1" pin="PGEC2"/>
+<pinref part="U1" gate="G$1" pin="RB11/PGEC2"/>
 <wire x1="83.82" y1="205.74" x2="86.36" y2="205.74" width="0.1524" layer="91"/>
 <label x="76.2" y="205.74" size="1.778" layer="95"/>
@@
 </segment>
 <segment>
-<pinref part="U1" gate="G$1" pin="SDI2/RA7"/>
+<pinref part="U1" gate="G$1" pin="OC5/SDI2/RA7"/>
 <wire x1="198.12" y1="198.12" x2="195.58" y2="198.12" width="0.1524" layer="91"/>
 <label x="200.66" y="198.12" size="1.778" layer="95"/>
@@
 </segment>
 <segment>
-<pinref part="U1" gate="G$1" pin="RB12/AN12/OC2B/DAC1OUT"/>
+<pinref part="U1" gate="G$1" pin="RB12/AN12/IC3/DAC1OUT"/>
 <wire x1="198.12" y1="215.9" x2="195.58" y2="215.9" width="0.1524" layer="91"/>
 <label x="200.66" y="215.9" size="1.778" layer="95"/>

Commit message: rev0
Parts:
- C12: MANUF (none) -> Murata; PN (none) -> GRM31CR61E226ME15L
Connections:
- net BRAKE_SW: now also U1.CN0/RA4; no longer U1.RA4/AN16
- net ENC_A: now also U1.CN2/RA0; no longer U1.RA0/AN0/C3INC
- net ENC_B: now also U1.CN3/RA1; no longer U1.RA1/AN1
- net ENC_SW: now also U1.CN7/RB3; no longer U1.RB3/AN5/OA1OUT/C2INC
- net RUN_SW: now also U1.CN27/RB5; no longer U1.SCK2/RB5
Other:
- note added: "add LCD"
- note added: "connector for the bridge"
- note added: "d2pak bridge"
- note added: "look at LT1676"
- note added: "rev.pol.prot sot"
- note added: "todo:"
Changed lines of the file:
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@@
 <part name="R4" library="ch_passive" deviceset="RESISTOR" device="-0603" value="10K"/>
 <part name="GND12" library="ch_passive" deviceset="GND" device=""/>
-<part name="C12" library="ch_passive" deviceset="CAP" device="1206" value="22uF"/>
+<part name="C12" library="ch_passive" deviceset="CAP" device="1206" value="22uF">
+<attribute name="MANUF" value="Murata"/>
+<attribute name="PN" value="GRM31CR61E226ME15L"/>
+</part>
 <part name="C13" library="ch_passive" deviceset="C" device="-0603" value="0.1"/>
 <part name="C14" library="ch_passive" deviceset="C" device="-0603" value="0.1"/>
@@
 <text x="48.26" y="66.04" size="2.54" layer="97">VBAT 7-50V</text>
 <text x="416.56" y="7.62" size="2.54" layer="97">0</text>
+<text x="48.26" y="60.96" size="1.778" layer="97">look at LT1676</text>
+<text x="38.1" y="60.96" size="1.778" layer="97">todo:</text>
+<text x="48.26" y="55.88" size="1.778" layer="97">add LCD</text>
+<text x="48.26" y="50.8" size="1.778" layer="97">connector for the bridge</text>
+<text x="48.26" y="45.72" size="1.778" layer="97">d2pak bridge</text>
+<text x="48.26" y="40.64" size="1.778" layer="97">rev.pol.prot sot</text>
 </plain>
 <instances>
@@
 <attribute name="NAME" x="302.26" y="226.06" size="1.778" layer="95"/>
 <attribute name="VALUE" x="302.26" y="223.52" size="1.778" layer="96"/>
+<attribute name="MANUF" x="307.34" y="220.98" size="1.778" layer="96" rot="R90" display="off"/>
+<attribute name="PN" x="307.34" y="220.98" size="1.778" layer="96" rot="R90" display="off"/>
 </instance>
 <instance part="C13" gate="G$1" x="307.34" y="205.74" smashed="yes" rot="R270">
@@
 </segment>
 <segment>
-<pinref part="U1" gate="G$1" pin="RA0/AN0/C3INC"/>
+<pinref part="U1" gate="G$1" pin="CN2/RA0"/>
 <wire x1="198.12" y1="175.26" x2="195.58" y2="175.26" width="0.1524" layer="91"/>
 <label x="200.66" y="175.26" size="1.778" layer="95"/>
@@
 </segment>
 <segment>
-<pinref part="U1" gate="G$1" pin="RA1/AN1"/>
+<pinref part="U1" gate="G$1" pin="CN3/RA1"/>
 <wire x1="198.12" y1="180.34" x2="195.58" y2="180.34" width="0.1524" layer="91"/>
 <label x="200.66" y="180.34" size="1.778" layer="95"/>
@@
 </segment>
 <segment>
-<pinref part="U1" gate="G$1" pin="RB3/AN5/OA1OUT/C2INC"/>
+<pinref part="U1" gate="G$1" pin="CN7/RB3"/>
 <wire x1="198.12" y1="187.96" x2="195.58" y2="187.96" width="0.1524" layer="91"/>
 <label x="200.66" y="187.96" size="1.778" layer="95"/>
@@
 </segment>
 <segment>
-<pinref part="U1" gate="G$1" pin="SCK2/RB5"/>
+<pinref part="U1" gate="G$1" pin="CN27/RB5"/>
 <wire x1="198.12" y1="195.58" x2="195.58" y2="195.58" width="0.1524" layer="91"/>
 <label x="200.66" y="195.58" size="1.778" layer="95"/>
@@
 </segment>
 <segment>
-<pinref part="U1" gate="G$1" pin="RA4/AN16"/>
+<pinref part="U1" gate="G$1" pin="CN0/RA4"/>
 <wire x1="198.12" y1="182.88" x2="195.58" y2="182.88" width="0.1524" layer="91"/>
 <label x="200.66" y="182.88" size="1.778" layer="95"/>
